Commit message: feat: add pointcloud as sensor data

File: bebop_gazebo/urdf/bebop_base.urdf.xacro (robot description, xacro)
@@ -13,4 +13,11 @@
   <!-- Main quadrotor link -->
   <xacro:macro name="bebop_base_macro">
+    <link name="world"/>
+    <joint name='virtual_joint' type='floating'>
+      <origin xyz="0 0 0.0" rpy="0 0 0" />
+      <parent link="world"/>
+      <child link="base_link"/>
+      <axis xyz="0 0 0"/>
+    </joint>
     <link name="base_link">
       <inertial>
@@ -73,5 +80,5 @@
     </joint>
     <link name='lidar_link'>
-      <!-- <origin xyz="0 0 0.1" rpy="0 0 0" /> -->
+      <origin xyz="0 0 0.1" rpy="0 0 0" />
       <inertial>
         <mass value="1e-5" />
@@ -115,7 +122,9 @@
             </range>
           </ray>
-          <plugin name="laser_controller" filename="libgazebo_ros_ray_sensor.so">
-              <output_type>sensor_msgs/LaserScan</output_type>
-              <frame_name>lidar_link</frame_name>
+          <plugin name="laser_controller" filename="libgazebo_ros_laser.so">
+              <alwaysOn>true</alwaysOn>
+              <updateRate>15.0</updateRate>
+              <topicName>scan</topicName>
+              <frameName>world</frameName>
           </plugin>
       </sensor>
@@ -124,4 +133,7 @@
       <material>Gazebo/Black</material>
     </gazebo>
+    <gazebo reference="base_link">
+      <plugin name="uav_control_plugin" filename="/home/shaswat/ros_ws/devel/lib/libplugin.so"/>
+    </gazebo>
   </xacro:macro>
 </robot>
